Commit message: updating files

File: urdf/materials.urdf.xacro (robot description, xacro)
@@ -1,51 +1,83 @@
 <?xml version="1.0"?>
-<robot>
-    <material name="black">
-    <color rgba="0.2 0.2 0.2 1.0"/>
-    </material>
-    <material name="orange">
-    <color rgba="1.0 0.55 0.0 1.0"/>
-    </material>
-    <material name="grey20">
-        <color rgba="0.2 0.2 0.2 1.0"/>
-    </material>
-    <material name="grey25">
-        <color rgba="0.25 0.25 0.25 1.0"/>
-    </material>
-    <material name="grey30">
-        <color rgba="0.3 0.3 0.3 1.0"/>
-    </material>
-    <material name="grey40">
-        <color rgba="0.4 0.4 0.4 1.0"/>
-    </material>
-    <material name="grey50">
-        <color rgba="0.5 0.5 0.5 1.0"/>
-    </material>
-    <material name="grey60">
-        <color rgba="0.6 0.6 0.6 1.0"/>
-    </material>
-    <material name="grey70">
-        <color rgba="0.7 0.7 0.7 1.0"/>
-    </material>
-    <material name="grey75">
-        <color rgba="0.75 0.75 0.75 1.0"/>
-    </material>
-    <material name="grey">
-        <color rgba="0.5 0.5 0.5 1.0"/>
-    </material>
-    <material name="red">
-        <color rgba="0.8 0.0 0.0 1.0"/>
-    </material>
-    <material name="white">
-        <color rgba="1.0 1.0 1.0 1.0"/>
-    </material>
-    <material name="blue">
-        <color rgba="0.0 0.0 0.8 1.0"/>
-    </material>
-    <material name="green">
-        <color rgba="0.0 0.8 0.0 1.0"/>
-    </material>
-    <material name="lightblue">
-        <color rgba="0.55 0.75 0.9 10"/>
-    </material>
+<robot xmlns:xacro="http://www.ros.org/wiki/xacro">
+    <macro name="color_black">
+        <material name="black">
+            <color rgba="0.2 0.2 0.2 1.0"/>
+        </material>
+    </macro>
+    <macro name="color_orange">
+        <material name="orange">
+            <color rgba="1.0 0.55 0.0 1.0"/>
+        </material>
+    </macro>
+    <macro name="color_grey20">
+        <material name="grey20">
+            <color rgba="0.2 0.2 0.2 1.0"/>
+        </material>
+    </macro>
+    <macro name="color_grey25">
+        <material name="grey25">
+            <color rgba="0.25 0.25 0.25 1.0"/>
+        </material>
+    </macro>
+    <macro name="color_grey30">
+        <material name="grey30">
+            <color rgba="0.3 0.3 0.3 1.0"/>
+        </material>
+    </macro>
+    <macro name="color_grey40">
+        <material name="grey40">
+            <color rgba="0.4 0.4 0.4 1.0"/>
+        </material>
+    </macro>
+    <macro name="color_grey50">
+        <material name="grey50">
+            <color rgba="0.5 0.5 0.5 1.0"/>
+        </material>
+    </macro>
+    <macro name="color_grey60">
+        <material name="grey60">
+            <color rgba="0.6 0.6 0.6 1.0"/>
+        </material>
+    </macro>
+    <macro name="color_grey70">
+        <material name="grey70">
+            <color rgba="0.7 0.7 0.7 1.0"/>
+        </material>
+    </macro>
+    <macro name="color_grey75">
+        <material name="grey75">
+            <color rgba="0.75 0.75 0.75 1.0"/>
+        </material>
+    </macro>
+    <macro name="color_grey">
+        <material name="grey">
+            <color rgba="0.5 0.5 0.5 1.0"/>
+        </material>
+    </macro>
+    <macro name="color_red">
+        <material name="red">
+            <color rgba="0.8 0.0 0.0 1.0"/>
+        </material>
+    </macro>
+    <macro name="color_white">
+        <material name="white">
+            <color rgba="1.0 1.0 1.0 1.0"/>
+        </material>
+    </macro>
+    <macro name="color_blue">
+        <material name="blue">
+            <color rgba="0.0 0.0 0.8 1.0"/>
+        </material>
+    </macro>
+    <macro name="color_green">
+        <material name="green">
+            <color rgba="0.0 0.8 0.0 1.0"/>
+        </material>
+    </macro>
+    <macro name="color_lightblue">
+        <material name="lightblue">
+            <color rgba="0.55 0.75 0.9 1.0"/>
+        </material>
+    </macro>
 </robot>

File: urdf/stikklar.urdf (robot description, URDF)
Before this commit: robot stikklar, 19 links, 18 joints
Links:
- added link lf_wheel_link; visual cylinder length=0.005 radius=0.026
- added link lr_wheel_link; visual cylinder length=0.005 radius=0.026
- added link neck_tilt_link, mass 0.00001; collision box size=0.025 0.0485 0.0375; visual mesh filename=package://stikklar_description/meshes/F2.stl scale=0.001 0.001 0.001
- added link rf_wheel_link; visual cylinder length=0.005 radius=0.026
- added link rr_wheel_link; visual cylinder length=0.005 radius=0.026
- link lf_coxa_bone_link: geometry collision box size=0.025 0.0485 0.0375; collision box size=0.028 0.0485 0.008
- link lf_femur_bone_link: geometry collision box size=0.028 0.0485 0.008; collision box size=0.028 0.0485 0.008
- link lf_tibia_bone_link: geometry collision box size=0.02 0.02 0.04; collision box size=0.02 0.02 0.1
- link lr_coxa_bone_link: geometry collision box size=0.025 0.0485 0.0375; collision box size=0.028 0.0485 0.008
- link lr_femur_bone_link: geometry collision box size=0.028 0.0485 0.008; collision box size=0.028 0.0485 0.008
- link lr_tibia_bone_link: geometry collision box size=0.02 0.02 0.04; collision box size=0.02 0.02 0.1
- link neck_pan_link: geometry collision box size=0.028 0.0485 0.008; collision box size=0.032 0.040 0.0501
- link rf_coxa_bone_link: geometry collision box size=0.025 0.0485 0.0375; collision box size=0.028 0.0485 0.008
- link rf_femur_bone_link: geometry collision box size=0.028 0.0485 0.008; collision box size=0.028 0.0485 0.008
- link rf_tibia_bone_link: geometry collision box size=0.02 0.02 0.04; collision box size=0.02 0.02 0.1
- link rr_coxa_bone_link: geometry collision box size=0.025 0.0485 0.0375; collision box size=0.028 0.0485 0.008
- link rr_femur_bone_link: geometry collision box size=0.028 0.0485 0.008; collision box size=0.028 0.0485 0.008
- link rr_tibia_bone_link: geometry collision box size=0.02 0.02 0.04; collision box size=0.02 0.02 0.1
Joints:
- added joint lf_wheel_joint: type continuous, parent lf_tibia_bone_link, child lf_wheel_link, origin xyz=0 -0.05 -0.153 rpy=0 1.57079632679 0, axis 0 1 0
- added joint lr_wheel_joint: type continuous, parent lr_tibia_bone_link, child lr_wheel_link, origin xyz=0 -0.05 -0.153 rpy=0 1.57079632679 0, axis 0 1 0
- added joint neck_tilt_joint: type revolute, parent neck_pan_link, child neck_tilt_link, origin xyz=0 0.038 0 rpy=3.14159265359 0 0, axis 1 0 0, limit lower=-1.5707 upper=1.5707 effort=30 velocity=100
- added joint rf_wheel_joint: type continuous, parent rf_tibia_bone_link, child rf_wheel_link, origin xyz=0 -0.05 -0.153 rpy=0 1.57079632679 0, axis 0 1 0
- added joint rr_wheel_joint: type continuous, parent rr_tibia_bone_link, child rr_wheel_link, origin xyz=0 -0.05 -0.153 rpy=0 1.57079632679 0, axis 0 1 0
- joint lf_shoulder_joint: origin xyz=0.1 0.1 0 rpy=1.57079632679 0 -0.7853981634 -> xyz=-0.1 0.1 0 rpy=1.57079632679 0 0.7853981634
- joint lf_tibia_bone_joint: limit lower=-1.78964425253 upper=1.72828502102 effort=30 velocity=100 -> lower=-2.443 upper=2.443 effort=30 velocity=100
- joint lr_shoulder_joint: origin xyz=-0.1 0.1 0 rpy=1.57079632679 0 0.7853981634 -> xyz=-0.1 -0.1 0 rpy=1.57079632679 0 2.35619449019
- joint lr_tibia_bone_joint: limit lower=-1.78964425253 upper=1.72828502102 effort=30 velocity=100 -> lower=-2.443 upper=2.443 effort=30 velocity=100
- joint neck_base_joint: origin xyz=0 0 0.0685 rpy=1.57079632679 0 0 -> xyz=0 0 0.0665 rpy=1.57079632679 0 0
- joint neck_pan_joint: axis 0 1 0 -> 0 -1 0; origin xyz=0 0 -0.082 rpy=0 0 0 -> xyz=0 0 0 rpy=0 0 0
- joint rf_shoulder_joint: origin xyz=0.1 -0.1 0 rpy=1.57079632679 0 -2.35619449019 -> xyz=0.1 0.1 0 rpy=1.57079632679 0 -0.7853981634
- joint rf_tibia_bone_joint: limit lower=-1.78964425253 upper=1.72828502102 effort=30 velocity=100 -> lower=-2.443 upper=2.443 effort=30 velocity=100
- joint rr_shoulder_joint: origin xyz=-0.1 -0.1 0 rpy=1.57079632679 0 2.35619449019 -> xyz=0.1 -0.1 0 rpy=1.57079632679 0 -2.35619449019
- joint rr_tibia_bone_joint: limit lower=-1.78964425253 upper=1.72828502102 effort=30 velocity=100 -> lower=-2.443 upper=2.443 effort=30 velocity=100

File: urdf/stikklar.urdf.xacro (robot description, xacro)
@@ -1,10 +1,10 @@
 <?xml version="1.0"?>
 <robot xmlns:xacro="http://www.ros.org/wiki/xacro" name="stikklar">
-	<xacro:include filename="/home/viki/catkin_ws/src/stikklar_description/urdf/stikklar_parts.urdf.xacro" />
-	<xacro:base size="0.14 0.14 0.055" color="grey30" />
-	<xacro:stikklar_leg parent="base" name="lf" xyz="${HALFBASE} ${HALFBASE} 0" rpy="${MPI2} 0 ${-MPI4}" />
-	<xacro:stikklar_leg parent="base" name="rf" xyz="${HALFBASE} -${HALFBASE} 0"  rpy="${MPI2} 0 ${MPI4-MPI}" />
-	<xacro:stikklar_leg parent="base" name="lr" xyz="-${HALFBASE} ${HALFBASE} 0"  rpy="${MPI2} 0 ${MPI4}" />
-	<xacro:stikklar_leg parent="base" name="rr" xyz="-${HALFBASE} -${HALFBASE} 0" rpy="${MPI2} 0 ${MPI-MPI4}" />
+	<xacro:include filename="$(find stikklar_description)/urdf/stikklar_parts.urdf.xacro" />
+	<xacro:base size="0.14 0.14 0.055" />
+	<xacro:stikklar_leg parent="base" name="lf" xyz="-${HALFBASE} ${HALFBASE} 0"  rpy="${MPI2} 0 ${MPI4}"     side="-1" />
+	<xacro:stikklar_leg parent="base" name="lr" xyz="-${HALFBASE} -${HALFBASE} 0" rpy="${MPI2} 0 ${MPI-MPI4}" side="1"  />
+	<xacro:stikklar_leg parent="base" name="rr" xyz="${HALFBASE} -${HALFBASE} 0"  rpy="${MPI2} 0 ${MPI4-MPI}" side="-1"  />
+	<xacro:stikklar_leg parent="base" name="rf" xyz="${HALFBASE} ${HALFBASE} 0"   rpy="${MPI2} 0 ${-MPI4}"    side="1"  />
 	<xacro:stikklar_turret parent="base" />
 </robot>

File: urdf/stikklar_config.urdf.xacro (robot description, xacro)
@@ -92,9 +92,9 @@
 	<property name="MIN_RAD_COXA" value="-2.3111977204143663" />
 	<property name="MIN_RAD_FEMUR" value="-1.7896442525332481" />
-	<property name="MIN_RAD_TIBIA" value="-2.132233295161041" />
+	<property name="MIN_RAD_TIBIA" value="-2.443" />
 	<!-- max servo values: 	coxa=960 femur=850 tibia=1005-->
 	<property name="MAX_RAD_COXA" value="2.2907446432425576" />
 	<property name="MAX_RAD_FEMUR" value="1.7282850210178222" />
-	<property name="MAX_RAD_TIBIA" value="2.5208417614254039" />
+	<property name="MAX_RAD_TIBIA" value="2.443" />
 	<!-- neutral servo values: 	coxa=364 femur=512 tibia=742-->
 	<property name="NEUTRAL_RAD_COXA" value="-0.75676385535691648" />

File: urdf/stikklar_parts.urdf.xacro (robot description, xacro)
@@ -2,12 +2,5 @@
 <robot xmlns:xacro="http://www.ros.org/wiki/xacro">
     <xacro:include filename="stikklar_config.urdf.xacro" />
-    <macro name="collision_box" params="xyz rpy size">
-        <collision>
-            <origin xyz="${xyz}" rpy="${rpy}" />
-            <geometry>
-                <box size="${size}" />
-            </geometry>
-        </collision>
-    </macro>
+    <xacro:include filename="materials.urdf.xacro" />
     <macro name="inertia_default">
         <inertial>
@@ -17,5 +10,5 @@
         </inertial>
     </macro>
-    <macro name="visual_box" params="color size xyz rpy">
+    <macro name="visual_box" params="size xyz rpy *color">
         <visual>
             <origin xyz="${xyz}" rpy="${rpy}" />
@@ -23,6 +16,14 @@
                 <box size="${size}" />
             </geometry>
-            <material name="${color}"/>
-        </visual>
+            <xacro:insert_block name="color" />
+        </visual>
+    </macro>
+    <macro name="collision_box" params="xyz rpy size">
+        <collision>
+            <origin xyz="${xyz}" rpy="${rpy}" />
+            <geometry>
+                <box size="${size}" />
+            </geometry>
+        </collision>
     </macro>
     <macro name="link_mesh" params="name mesh color box_xyz size scale">
@@ -39,11 +40,4 @@
         </link>
     </macro>
-    <macro name="link_box" params="name color size offset">
-        <link name="${name}_link">
-            <inertia_default />
-            <visual_box color="${color}" size="${size}" offset="${offset}" />
-            <collision_box xyz="${offset}" rpy="0 0 0" size="${size}" />
-        </link>
-    </macro>
     <macro name="joint_fixed" params="parent name xyz rpy">
         <joint name="${name}_joint" type="fixed">
@@ -72,5 +66,5 @@
             <origin xyz="${xyz}" rpy="${rpy}" />
             <geometry_ax12 />
-            <material name="grey30"/>
+            <color_black />
         </visual>
     </macro>
@@ -91,5 +85,5 @@
             <origin xyz="${xyz}" rpy="${rpy}" />
             <geometry_F1 />
-            <material name="grey60"/>
+            <color_grey60 />
         </visual>
     </macro>
@@ -110,5 +104,5 @@
             <origin xyz="${xyz}" rpy="${rpy}" />
             <geometry_F2 />
-            <material name="grey60"/>
+            <color_grey60 />
         </visual>
     </macro>
@@ -128,10 +122,10 @@
         <visual>
             <origin xyz="${xyz}" rpy="${rpy}" />
-            <material name="grey60"/>
+            <color_grey60 />
             <geometry_F3 />
         </visual>
     </macro>
     <macro name="collision_F3" params="xyz rpy">
-        <collision_box xyz="${xyz}" rpy="${rpy}" size="0.028 0.0485 0.065" />
+        <collision_box xyz="${xyz}" rpy="${rpy}" size="0.028 0.0485 0.008" />
     </macro>
     <macro name="part_F3" params="xyz rpy">
@@ -147,5 +141,6 @@
         <visual>
             <origin xyz="${xyz}" rpy="${rpy}" />
-            <material name="grey60"/>
+            <!-- <material name="green"/> -->
+            <color_grey60 />
             <geometry_F4 />
         </visual>
@@ -158,28 +153,19 @@
         <visual_F4 xyz="${xyz}" rpy="${rpy}" />
     </macro>
-    <macro name="geometry_F4">
-        <geometry>
-            <mesh filename="package://${PACKAGE}/meshes/F4.stl" scale="${M_SCALE_3}"/>
-        </geometry>
-    </macro>
-    <macro name="visual_F4" params="xyz rpy">
-        <visual>
-            <origin xyz="${xyz}" rpy="${rpy}" />
-            <material name="grey60"/>
-            <geometry_F4 />
-        </visual>
-    </macro>
-    <macro name="collision_F4" params="xyz rpy">
-        <collision_box xyz="${xyz}" rpy="${rpy}" size="0.028 0.0485 0.065" />
-    </macro>
-    <macro name="part_box" params="xyz rpy size color">
+    <macro name="part_box" params="xyz rpy size *color">
         <collision_box xyz="${xyz}" rpy="${rpy}" size="${size}" />
-        <visual_box xyz="${xyz}" rpy="${rpy}" size="${size}" color="${color}" />
+        <visual_box xyz="${xyz}" rpy="${rpy}" size="${size}">
+            <xacro:insert_block name="color" />
+        </visual_box>
     </macro>
     <macro name="part_tibia_bone" params="xyz rpy">
-        <part_box xyz="${xyz}" rpy="${rpy}" size="0.02 0.02 0.1" color="grey70" />
+        <part_box xyz="${xyz}" rpy="${rpy}" size="0.02 0.02 0.1">
+            <color_grey50 />
+        </part_box>
     </macro>
     <macro name="part_tibia_bone_spacer" params="xyz rpy">
-        <part_box xyz="${xyz}" rpy="${rpy}" size="0.02 0.02 0.04" color="grey70" />
+        <part_box xyz="${xyz}" rpy="${rpy}" size="0.02 0.02 0.04">
+            <color_grey50 />
+        </part_box>
     </macro>
     <!-- link+join+composite visuals and collisions -->
@@ -201,11 +187,11 @@
             vel="100" llimit="${MIN_RAD_COXA}" ulimit="${MAX_RAD_COXA}" axis="0 1 0" />
     </macro>
-    <macro name="femur_bone" params="parent name">
+    <macro name="femur_bone" params="parent name side">
         <link name="${name}_link">
             <inertia_default />
             <part_ax12 xyz="0 0 0" rpy="0 0 ${MPI2}"/>
             <part_F3 xyz="0 0 -0.0415" rpy="0 ${MPI} 0"/>
-            <part_F3 xyz="0.008 0 -0.0415" rpy="0 0 0"/>
-            <part_ax12 xyz="0.008 0 -${L_FEMUR}" rpy="${MPI} 0 -${MPI2}"/>
+            <part_F3 xyz="${side*0.008} 0 -0.0415" rpy="0 0 0"/>
+            <part_ax12 xyz="${side*0.008} 0 -${L_FEMUR}" rpy="${MPI} 0 -${MPI2}"/>
         </link>
         <joint_revolute name="${name}" parent="${parent}" xyz="0 0 -${L_COXA}" rpy="0 0 0"
@@ -215,18 +201,18 @@
     <property name="TIBIA_AY" value="0.015" />
     <property name="TIBIA_AZ" value="0.0755" />
-    <property name="F3T" value="0.04772" />
-    <property name="AX12T" value="0.06328" />
-    <macro name="tibia_bone" params="parent name">
-        <link name="${name}_link">
-            <inertia_default />
-            <part_F4 xyz="${TIBIA_AX} 0 0" rpy="0 ${MPI} ${MPI2}" />
-            <part_F1 xyz="${TIBIA_AX} ${-TIBIA_AY} ${-TIBIA_AZ}" rpy="-${MPI2} 0 ${MPI2}" />
-            <part_tibia_bone xyz="0.018 ${-TIBIA_AX-0.0318} ${-TIBIA_AZ-0.0318}" rpy="-${MPI4} 0 0" />
-            <part_tibia_bone_spacer xyz="-0.0025 ${-TIBIA_AY-0.00707} ${-TIBIA_AZ-0.00707}" rpy="-${MPI4} 0 0" />
-            <part_F3 xyz="0.0235 ${-TIBIA_AX-F3T+0.00707} ${-TIBIA_AZ-F3T-0.00707}" rpy="0 -${MPI4} ${MPI2}" />
-            <part_ax12 xyz="0.0235 ${-TIBIA_AX-AX12T+0.0205} ${-TIBIA_AZ-AX12T-0.0205}" rpy="${MPI} -${MPI4} -${MPI2}" />
+    <property name="F3T" value="0.04072" />
+    <property name="AX12T" value="0.0566" />
+    <macro name="tibia_bone" params="parent name side">
+        <link name="${name}_link">
+            <inertia_default />
+            <part_F4 xyz="${side*TIBIA_AX} 0 0" rpy="0 ${MPI} ${MPI2}" />
+            <part_F1 xyz="${side*TIBIA_AX} ${-TIBIA_AY} ${-TIBIA_AZ}" rpy="-${MPI2} 0 ${MPI2}" />
+            <part_tibia_bone xyz="${side*0.018} ${-TIBIA_AY-0.0282} ${-TIBIA_AZ-0.0282}" rpy="-${MPI4} 0 0" />
+            <part_tibia_bone_spacer xyz="${side*-0.0025} ${-TIBIA_AY-0.00707} ${-TIBIA_AZ-0.00707}" rpy="-${MPI4} 0 0" />
+            <part_F3 xyz="${side*0.0235} ${-TIBIA_AY-F3T+0.00707} ${-TIBIA_AZ-F3T-0.00707}" rpy="0 -${MPI4} ${MPI2}" />
+            <part_ax12 xyz="${side*0.0235} ${-TIBIA_AY-AX12T+0.0205} ${-TIBIA_AZ-AX12T-0.0205}" rpy="${MPI} -${MPI4} -${MPI2}" />
         </link>
         <joint_revolute name="${name}" parent="${parent}" xyz="0 0 -${L_FEMUR}" rpy="0 0 0"
-            vel="100" llimit="${MIN_RAD_FEMUR}" ulimit="${MAX_RAD_FEMUR}" axis="${VLEFT}" />
+            vel="100" llimit="${MIN_RAD_TIBIA}" ulimit="${MAX_RAD_TIBIA}" axis="${VLEFT}" />
     </macro>
     <macro name="neck_base" params="name parent">
@@ -245,40 +231,47 @@
         </link>
         <joint_revolute name="${name}" parent="${parent}" xyz="0 0 0" rpy="0 0 0"
-            vel="100" llimit="${MIN_PAN}" ulimit="${MAX_PAN}" axis="0 1 0" />
-    </macro>
-    <!--macro name="neck_tilt" params="name parent">
-        <link name="${name}_link">
-            <inertia_default />
-        </link>
-    </macro-->
-    <macro name="wheel">
-        <link name="b_l_wheel">
+            vel="100" llimit="${MIN_PAN}" ulimit="${MAX_PAN}" axis="0 -1 0" />
+    </macro>
+    <macro name="neck_tilt" params="name parent">
+        <link name="${name}_link">
+            <inertia_default />
+            <part_F2 xyz="0 0 0" rpy="${MPI2} ${MPI2} 0"/>
+        </link>
+        <joint_revolute name="${name}" parent="${parent}" xyz="0 0.038 0" rpy="${MPI} 0 0"
+            vel="100" llimit="${MIN_TILT}" ulimit="${MAX_TILT}" axis="1 0 0" />
+    </macro>
+    <macro name="wheel" params="parent name">
+        <link name="${name}_link">
             <visual>
                 <origin xyz="0 0 0" rpy="0 0 0" />
                 <geometry>
-                    <cylinder length="0.007" radius="0.026" />
+                    <cylinder length="0.005" radius="0.026" />
                 </geometry>
+                <color_grey30 />
             </visual>
         </link>
-        <joint name="joint_b_l_wheel" type="continuous">
-            <parent link="base_link"/>
-            <child link="b_l_wheel"/>
-            <origin xyz="-0.25 0.30 0" rpy="0 0 0" />
+        <joint name="${name}_joint" type="continuous">
+            <parent link="${parent}_link"/>
+            <child link="${name}_link"/>
+            <origin xyz="0 -0.05 -0.153" rpy="0 ${MPI2} 0" />
             <axis xyz="0 1 0" rpy="0 0 0" />
         </joint>
     </macro>
-    <macro name="base" params="size color">
+    <macro name="base" params="size">
         <link name="base_link">
             <inertia_default />
-            <visual_box xyz="0 0 0" rpy="0 0 0" size="${size}" color="grey25" />
+            <visual_box xyz="0 0 0" rpy="0 0 0" size="${size}">
+                <color_black />
+            </visual_box>
             <collision_box xyz="0 0 0" rpy="0 0 0" size="${size}" />
         </link>
     </macro>
-    <macro name="stikklar_leg" params="parent name xyz rpy">
+    <macro name="stikklar_leg" params="parent name xyz rpy side">
         <!-- x=red y=green z=blue -->
         <shoulder parent="${parent}" name="${name}_shoulder" xyz="${xyz}" rpy="${rpy}" />
         <coxa_bone parent="${name}_shoulder" name="${name}_coxa_bone" />
-        <femur_bone parent="${name}_coxa_bone" name="${name}_femur_bone" />
-        <tibia_bone parent="${name}_femur_bone" name="${name}_tibia_bone" />
+        <femur_bone parent="${name}_coxa_bone" name="${name}_femur_bone" side="${side}" />
+        <tibia_bone parent="${name}_femur_bone" name="${name}_tibia_bone" side="${side}" />
+        <wheel parent="${name}_tibia_bone" name="${name}_wheel" />
     </macro>
     <macro name="stikklar_turret" params="parent">
@@ -287,4 +280,3 @@
         <neck_tilt parent="neck_pan" name="neck_tilt" />
     </macro>
-    <xacro:include filename="materials.urdf.xacro" />
 </robot>
