Commit message: updating urdf scripts, adding head, fixing wheel axis

File: urdf/stikklar_parts.urdf.xacro (robot description, xacro)
@@ -237,4 +237,14 @@
             <inertia_default />
             <part_F2 xyz="0 0 0" rpy="${MPI2} ${MPI2} 0"/>
+            <part_box xyz="0 -0.076 0" rpy="0 0 0" size="0.065 0.1 0.03">
+                <color_grey70 />
+            </part_box>
+            <visual>
+                <origin xyz="0.013 -0.081 0.015" rpy="0 0 0" />
+                <geometry>
+                    <cylinder length="0.002" radius="0.004" />
+                </geometry>
+                <color_black />
+            </visual>
         </link>
         <joint_revolute name="${name}" parent="${parent}" xyz="0 0.038 0" rpy="${MPI} 0 0"
@@ -255,5 +265,5 @@
             <child link="${name}_link"/>
             <origin xyz="0 -0.05 -0.153" rpy="0 ${MPI2} 0" />
-            <axis xyz="0 1 0" rpy="0 0 0" />
+            <axis xyz="0 0 1" rpy="0 0 0" />
         </joint>
     </macro>

Commit message: latest updates

File: urdf/stikklar_parts.urdf.xacro (robot description, xacro)
@@ -3,4 +3,8 @@
     <xacro:include filename="stikklar_config.urdf.xacro" />
     <xacro:include filename="materials.urdf.xacro" />
+    <xacro:include filename="gazebo.urdf.xacro" />
+    <macro name="to_vec" params="src">
+        <property name="vec" value="${map(float, src.split())}" />
+    </macro>
     <macro name="inertia_default">
         <inertial>
@@ -70,5 +74,6 @@
     </macro>
     <macro name="collision_ax12" params="xyz rpy">
-        <collision_box xyz="${xyz}" rpy="0 0 0" size="0.032 0.040 0.0501" />
+        <property name="vec" value="${map(float, xyz.split())}" />
+        <collision_box xyz="${vec[0]} ${vec[1]} ${vec[2]-0.013}" rpy="${rpy}" size="0.032 0.038 0.049" />
     </macro>
     <macro name="part_ax12" params="xyz rpy">
@@ -108,5 +113,6 @@
     </macro>
     <macro name="collision_F2" params="xyz rpy">
-        <collision_box xyz="${xyz}" rpy="${rpy}" size="0.025 0.0485 0.0375" />
+        <property name="vec" value="${map(float, xyz.split())}" />
+        <collision_box xyz="${vec[0]} ${vec[1]} ${vec[2]+0.008}"  rpy="${rpy}" size="0.025 0.0485 0.0375" />
     </macro>
     <macro name="part_F2" params="xyz rpy">
@@ -127,5 +133,6 @@
     </macro>
     <macro name="collision_F3" params="xyz rpy">
-        <collision_box xyz="${xyz}" rpy="${rpy}" size="0.028 0.0485 0.008" />
+        <property name="vec" value="${map(float, xyz.split())}" />
+        <collision_box xyz="${vec[0]} ${vec[1]} ${vec[2]+0.004}" rpy="${rpy}" size="0.025 0.038 0.008" />
     </macro>
     <macro name="part_F3" params="xyz rpy">
@@ -141,5 +148,4 @@
         <visual>
             <origin xyz="${xyz}" rpy="${rpy}" />
-            <!-- <material name="green"/> -->
             <color_grey60 />
             <geometry_F4 />
@@ -147,5 +153,6 @@
     </macro>
     <macro name="collision_F4" params="xyz rpy">
-        <collision_box xyz="${xyz}" rpy="${rpy}" size="0.028 0.0485 0.065" />
+        <property name="vec" value="${map(float, xyz.split())}" />
+        <collision_box xyz="${vec[0]+0.0} ${vec[1]+0.0} ${vec[2]+0.0}" rpy="${rpy}" size="0.028 0.0485 0.065" />
     </macro>
     <macro name="part_F4" params="xyz rpy">
@@ -197,4 +204,10 @@
         <joint_revolute name="${name}" parent="${parent}" xyz="0 0 -${L_COXA}" rpy="0 0 0"
             vel="100" llimit="${MIN_RAD_FEMUR}" ulimit="${MAX_RAD_FEMUR}" axis="${VLEFT}" />
+        <transmission name="${name}_transmission">
+            <type>transmission_interface/SimpleTransmission</type>
+            <actuator name="caster_front_left_motor" />
+            <joint name="caster_front_left_joint" />
+            <mechanicalReduction>1</mechanicalReduction>
+        </transmission>
     </macro>
     <property name="TIBIA_AX" value="0.008" />
