Commit message: updating gazebo definition. No inertial on base link and gazebo materials.

File: urdf/gazebo.urdf.xacro (robot description, xacro)
@@ -1,8 +1,39 @@
 <?xml version="1.0"?>
 <robot xmlns:xacro="http://www.ros.org/wiki/xacro">
+	<macro name="servo_transmission" params="name reduction">
+		<transmission name="${name}_transmission">
+			<type>transmission_interface/SimpleTransmission</type>
+			<joint name="${name}_joint">
+				<hardwareInterface>EffortJointInterface</hardwareInterface>
+			</joint>
+			<actuator name="${name}_motor">
+				<hardwareInterface>EffortJointInterface</hardwareInterface>
+				<mechanicalReduction>${reduction}</mechanicalReduction>
+			</actuator>
+		</transmission>
+	</macro>
+	<macro name="gazebo_color" params="ref color">
+		<gazebo reference="${ref}">
+			<material>Gazebo/${color}</material>
+		</gazebo>
+  	</macro>
 	<gazebo>
-	  <plugin name="gazebo_ros_control" filename="libgazebo_ros_control.so">
-	    <robotNamespace>/stikklar</robotNamespace>
-	  </plugin>
+		<plugin name="gazebo_ros_control" filename="libgazebo_ros_control.so">
+			<robotNamespace>/stikklar</robotNamespace>
+			<robotSimType>gazebo_ros_control/DefaultRobotHWSim</robotSimType>
+		</plugin>
 	</gazebo>
+	<gazebo_color ref="rr_tibia_bone_link" color="Grey" />
+	<gazebo_color ref="rf_tibia_bone_link" color="Grey" />
+	<gazebo_color ref="lr_tibia_bone_link" color="Grey" />
+	<gazebo_color ref="lf_tibia_bone_link" color="Grey" />
+	<gazebo_color ref="rr_femur_bone_link" color="Orange" />
+	<gazebo_color ref="rf_femur_bone_link" color="Orange" />
+	<gazebo_color ref="lr_femur_bone_link" color="Orange" />
+	<gazebo_color ref="lf_femur_bone_link" color="Orange" />
+	<gazebo_color ref="rr_coxa_bone_link" color="Blue" />
+	<gazebo_color ref="rf_coxa_bone_link" color="Blue" />
+	<gazebo_color ref="lr_coxa_bone_link" color="Blue" />
+	<gazebo_color ref="lf_coxa_bone_link" color="Blue" />
+	<gazebo_color ref="body_link" color="Green" />
 </robot>

File: urdf/stikklar.urdf.xacro (robot description, xacro)
@@ -2,5 +2,6 @@
 <robot xmlns:xacro="http://www.ros.org/wiki/xacro" name="stikklar">
 	<xacro:include filename="$(find stikklar_description)/urdf/stikklar_parts.urdf.xacro" />
-	<xacro:base size="0.14 0.14 0.055" />
+	<xacro:base />
+	<xacro:body parent="base" size="0.14 0.14 0.055" />
 	<xacro:stikklar_leg parent="base" name="lf" xyz="-${HALFBASE} ${HALFBASE} 0"  rpy="${MPI2} 0 ${MPI4}"     side="-1" />
 	<xacro:stikklar_leg parent="base" name="lr" xyz="-${HALFBASE} -${HALFBASE} 0" rpy="${MPI2} 0 ${MPI-MPI4}" side="1"  />

File: urdf/stikklar_parts.urdf.xacro (robot description, xacro)
@@ -7,7 +7,7 @@
         <property name="vec" value="${map(float, src.split())}" />
     </macro>
-    <macro name="inertia_default">
+    <macro name="inertia_default" params="mass">
         <inertial>
-            <mass value="0.00001" />
+            <mass value="${mass}" />
             <origin xyz="0 0 0" />
             <inertia ixx="1.0" ixy="0.0" ixz="0.0" iyy="1.0" iyz="0.0" izz="1.0" />
@@ -33,5 +33,5 @@
     <macro name="link_mesh" params="name mesh color box_xyz size scale">
         <link name="${name}_link">
-            <inertia_default />
+            <inertia_default mass="0.1" />
             <visual>
                 <origin xyz="0 0 0" rpy="0 0 0" />
@@ -60,5 +60,5 @@
         </joint>
     </macro>
-    <!-- atmic shapes, ax12, bioloids frames F1, F2, F3, F4 -->
+    <!-- atomic shapes, ax12, bioloids frames F1, F2, F3, F4 -->
     <macro name="geometry_ax12">
         <geometry>
@@ -179,5 +179,5 @@
     <macro name="shoulder" params="parent name xyz rpy">
         <link name="${name}_link">
-            <inertia_default />
+            <inertia_default mass="0.1" />
             <part_F4 xyz="0 0 0" rpy="0 0 0" />
         </link>
@@ -186,5 +186,6 @@
     <macro name="coxa_bone" params="parent name">
         <link name="${name}_link">
-            <inertia_default />
+            <gazebo_color ref="${name}_link" color="Green" />
+            <inertia_default mass="0.1" />
             <part_ax12 xyz="0 0 0" rpy="0 0 ${MPI}" />
             <part_F3 xyz="0 0 -0.0415" rpy="0 ${MPI} 0 "/>
@@ -193,8 +194,10 @@
         <joint_revolute name="${name}" parent="${parent}" xyz="0 0 0" rpy="0 0 0"
             vel="100" llimit="${MIN_RAD_COXA}" ulimit="${MAX_RAD_COXA}" axis="0 1 0" />
+        <servo_transmission name="${name}" reduction="1" />
     </macro>
     <macro name="femur_bone" params="parent name side">
         <link name="${name}_link">
-            <inertia_default />
+            <gazebo_color ref="${name}_link" color="Orange" />
+            <inertia_default mass="0.1" />
             <part_ax12 xyz="0 0 0" rpy="0 0 ${MPI2}"/>
             <part_F3 xyz="0 0 -0.0415" rpy="0 ${MPI} 0"/>
@@ -204,10 +207,5 @@
         <joint_revolute name="${name}" parent="${parent}" xyz="0 0 -${L_COXA}" rpy="0 0 0"
             vel="100" llimit="${MIN_RAD_FEMUR}" ulimit="${MAX_RAD_FEMUR}" axis="${VLEFT}" />
-        <transmission name="${name}_transmission">
-            <type>transmission_interface/SimpleTransmission</type>
-            <actuator name="caster_front_left_motor" />
-            <joint name="caster_front_left_joint" />
-            <mechanicalReduction>1</mechanicalReduction>
-        </transmission>
+        <servo_transmission name="${name}" reduction="1" />
     </macro>
     <property name="TIBIA_AX" value="0.008" />
@@ -218,5 +216,6 @@
     <macro name="tibia_bone" params="parent name side">
         <link name="${name}_link">
-            <inertia_default />
+            <gazebo_color ref="${name}_link" color="Blue" />
+            <inertia_default mass="0.1" />
             <part_F4 xyz="${side*TIBIA_AX} 0 0" rpy="0 ${MPI} ${MPI2}" />
             <part_F1 xyz="${side*TIBIA_AX} ${-TIBIA_AY} ${-TIBIA_AZ}" rpy="-${MPI2} 0 ${MPI2}" />
@@ -228,8 +227,9 @@
         <joint_revolute name="${name}" parent="${parent}" xyz="0 0 -${L_FEMUR}" rpy="0 0 0"
             vel="100" llimit="${MIN_RAD_TIBIA}" ulimit="${MAX_RAD_TIBIA}" axis="${VLEFT}" />
+        <servo_transmission name="${name}" reduction="1" />
     </macro>
     <macro name="neck_base" params="name parent">
         <link name="neck_base_link">
-            <inertia_default />
+            <inertia_default mass="0.1"  />
             <part_ax12 xyz="0 -0.023 0" rpy="0 0 0" />
         </link>
@@ -238,5 +238,5 @@
     <macro name="neck_pan" params="name parent">
         <link name="${name}_link">
-            <inertia_default />
+            <inertia_default mass="0.1"  />
             <part_F3 xyz="0 0 0" rpy="${MPI2} ${MPI2} 0"/>
             <part_ax12 xyz="0 0.04 0" rpy="-${MPI2} -${MPI2} 0" />
@@ -248,5 +248,5 @@
     <macro name="neck_tilt" params="name parent">
         <link name="${name}_link">
-            <inertia_default />
+            <inertia_default mass="0.1"  />
             <part_F2 xyz="0 0 0" rpy="${MPI2} ${MPI2} 0"/>
             <part_box xyz="0 -0.076 0" rpy="0 0 0" size="0.065 0.1 0.03">
@@ -281,7 +281,10 @@
         </joint>
     </macro>
-    <macro name="base" params="size">
-        <link name="base_link">
-            <inertia_default />
+    <macro name="base">
+        <link name="base_link"></link>
+    </macro>
+    <macro name="body" params="parent size">
+        <link name="body_link">
+            <inertia_default mass="0.3" />
             <visual_box xyz="0 0 0" rpy="0 0 0" size="${size}">
                 <color_black />
@@ -289,4 +292,5 @@
             <collision_box xyz="0 0 0" rpy="0 0 0" size="${size}" />
         </link>
+        <joint_fixed name="body" parent="${parent}" xyz="0 0 0" rpy="0 0 0" />
     </macro>
     <macro name="stikklar_leg" params="parent name xyz rpy side">
